Commit message: edit modle v0.0

File: ngws_description/urdf/ngws_v0.0.xacro (robot description, xacro)
@@ -4,5 +4,5 @@
   <!-- Constants for robot dimensions -->
   <xacro:property name="PI" value="3.1415926535897931"/>
-  <xacro:property name="mass" value="10" /> <!-- arbitrary value for mass -->
+  <xacro:property name="mass" value="30" /> <!-- arbitrary value for mass -->
   <xacro:property name="width" value="0.1" /> <!-- Square dimensions (widthxwidth) of beams -->
   <xacro:property name="height1" value="2" /> <!-- Link 1 -->
@@ -44,5 +44,5 @@
     </visual>
     <inertial>
-      <origin xyz="0 0 0.3" rpy="0 0 0"/>
+      <origin xyz="0 0 0" rpy="0 0 0"/>
       <mass value="${mass}"/>
       <inertia
@@ -58,4 +58,5 @@
     <parent link="base_link"/>
     <child link="wheel_FR_link"/>
+    <dynamics damping="0.05"/>
   </joint>
   <link name="wheel_FR_link">
@@ -74,5 +75,5 @@
     </visual>
     <inertial>
-      <mass value="2" />
+      <mass value="0.5" />
       <origin xyz="0 0 0" rpy="0 0 0"/>
         <inertia
@@ -88,4 +89,5 @@
     <parent link="base_link"/>
     <child link="wheel_FL_link"/>
+    <dynamics damping="0.05"/>
   </joint>
   <link name="wheel_FL_link">
@@ -104,5 +106,5 @@
     </visual>
     <inertial>
-      <mass value="2" />
+      <mass value="0.5" />
       <origin xyz="0 0 0" rpy="0 0 0"/>
         <inertia
@@ -118,4 +120,5 @@
     <parent link="base_link"/>
     <child link="wheel_BR_link"/>
+    <dynamics damping="0.05"/>
   </joint>
   <link name="wheel_BR_link">
@@ -134,5 +137,5 @@
     </visual>
     <inertial>
-      <mass value="2" />
+      <mass value="0.5" />
       <origin xyz="0 0 0" rpy="0 0 0"/>
         <inertia
@@ -148,4 +151,5 @@
     <parent link="base_link"/>
     <child link="wheel_BL_link"/>
+    <dynamics damping="0.05"/>
   </joint>
   <link name="wheel_BL_link">
@@ -164,5 +168,5 @@
     </visual>
     <inertial>
-      <mass value="2" />
+      <mass value="0.5" />
       <origin xyz="0 0 0" rpy="0 0 0"/>
         <inertia

Commit message: add omni model

File: ngws_description/urdf/ngws_v0.0.xacro (robot description, xacro)
@@ -12,5 +12,5 @@
   <xacro:property name="axel_offset" value="0.05" /> <!-- Space btw top of beam and the each joint -->
   <!-- Import all Gazebo-customization elements, including Gazebo colors -->
-  <xacro:include filename="$(find ngws_description)/urdf/gazebo/addon.gazebo" />
+  <xacro:include filename="$(find ngws_description)/urdf/gazebo/addon_v0.0.gazebo" />
   <!-- Import Rviz colors -->
   <xacro:include filename="$(find ngws_description)/urdf/materials/materials.xacro" />

File: ngws_description/urdf/ngws_v1.0.xacro (robot description, xacro)
@@ -4,15 +4,11 @@
   <!-- Constants for robot dimensions -->
   <xacro:property name="PI" value="3.1415926535897931"/>
-  <xacro:property name="mass" value="10" /> <!-- arbitrary value for mass -->
-  <xacro:property name="width" value="0.1" /> <!-- Square dimensions (widthxwidth) of beams -->
-  <xacro:property name="height1" value="2" /> <!-- Link 1 -->
-  <xacro:property name="height2" value="1" /> <!-- Link 2 -->
-  <xacro:property name="height3" value="1" /> <!-- Link 3 -->
-  <xacro:property name="camera_link" value="0.05" /> <!-- Size of square 'camera' box -->
-  <xacro:property name="axel_offset" value="0.05" /> <!-- Space btw top of beam and the each joint -->
+  <xacro:property name="mass" value="50" /> <!-- arbitrary value for mass -->
+  <xacro:property name="width" value="0.6" /> <!-- Square dimensions (widthxwidth) of beams -->
   <!-- Import all Gazebo-customization elements, including Gazebo colors -->
-  <xacro:include filename="$(find ngws_description)/urdf/gazebo/addon.gazebo" />
+  <xacro:include filename="$(find ngws_description)/urdf/gazebo/addon_v1.0.gazebo" />
   <!-- Import Rviz colors -->
   <xacro:include filename="$(find ngws_description)/urdf/materials/materials.xacro" />
+  <xacro:include filename="$(find ngws_description)/urdf/mecanum_wheel/mecanum_wheel.xacro" />
   <!-- Used for fixing robot to Gazebo 'base_link' -->
 <!--   <link name="world"/>
@@ -44,16 +40,99 @@
     </visual>
     <inertial>
-      <origin xyz="0 0 0.3" rpy="0 0 0"/>
+      <origin xyz="0 0 0.1" rpy="0 0 0"/>
       <mass value="${mass}"/>
       <inertia
-    ixx="${mass / 12.0 * (width*width + height1*height1)}" ixy="0.0" ixz="0.0"
-    iyy="${mass / 12.0 * (height1*height1 + width*width)}" iyz="0.0"
-    izz="${mass / 12.0 * (width*width + width*width)}"/>
+    ixx="${mass*0.083*2*width*width}" ixy="0.0" ixz="0.0"
+    iyy="${mass*0.083*2*width*width}" iyz="0.0"
+    izz="${mass*0.083*2*width*width}"/>
     </inertial>
   </link>
+  <!-- subwheel -->
+    <xacro:property name="wheel_mass" value="2"/>
+    <xacro:property name="main_radius" value="0.041"/>
+    <xacro:property name="caster" value="${PI*0.25}"/>
+    <xacro:property name="main_mesh_file" value="package://ngws_description/meshes/mecanum_wheel.stl"/>
+    <xacro:property name="main_mesh_file_rev" value="package://ngws_description/meshes/mecanum_wheel_r.stl"/>
+    <xacro:property name="sub_mesh_file" value="package://ngws_description/meshes/mecanum_miniwheel.stl"/>
+  <!-- FR -->
+  <xacro:mecanum_wheel_macro
+    name="wheel_FR"
+    parent_link="base_link"
+    mass="${wheel_mass}"
+    has_10_subwheel="true"
+    main_radius="${main_radius}"
+    caster="${caster}"
+    main_mesh_file="${main_mesh_file_rev}"
+    sub_mesh_file="${sub_mesh_file}"
+    mesh_scale="0.001"
+    x="0.3"
+    y="-0.3"
+    z="0.02"
+    R="0.0"
+    P="0.0"
+    Y="${PI/2}"
+    >
+  </xacro:mecanum_wheel_macro>
+<!-- FL -->
+  <xacro:mecanum_wheel_macro
+    name="wheel_FL"
+    parent_link="base_link"
+    mass="${wheel_mass}"
+    has_10_subwheel="true"
+    main_radius="${main_radius}"
+    caster="-${caster}"
+    main_mesh_file="${main_mesh_file}"
+    sub_mesh_file="${sub_mesh_file}"
+    mesh_scale="0.001"
+    x="0.3"
+    y="0.3"
+    z="0.02"
+    R="0.0"
+    P="0.0"
+    Y="${PI/2}"
+    >
+  </xacro:mecanum_wheel_macro>
+<!-- BR -->
+  <xacro:mecanum_wheel_macro
+    name="wheel_BR"
+    parent_link="base_link"
+    mass="${wheel_mass}"
+    has_10_subwheel="true"
+    main_radius="${main_radius}"
+    caster="-${caster}"
+    main_mesh_file="${main_mesh_file}"
+    sub_mesh_file="${sub_mesh_file}"
+    mesh_scale="0.001"
+    x="-0.3"
+    y="-0.3"
+    z="0.02"
+    R="0.0"
+    P="0.0"
+    Y="${PI/2}"
+    >
+  </xacro:mecanum_wheel_macro>
+<!-- BL -->
+  <xacro:mecanum_wheel_macro
+    name="wheel_BL"
+    parent_link="base_link"
+    mass="${wheel_mass}"
+    has_10_subwheel="true"
+    main_radius="${main_radius}"
+    caster="${caster}"
+    main_mesh_file="${main_mesh_file_rev}"
+    sub_mesh_file="${sub_mesh_file}"
+    mesh_scale="0.001"
+    x="-0.3"
+    y="0.3"
+    z="0.02"
+    R="0.0"
+    P="0.0"
+    Y="${PI/2}"
+    >
+  </xacro:mecanum_wheel_macro>
   <!-- Wheel FR -->
-  <joint name="wheel_FR_joint" type="continuous">
+  <!-- <joint name="wheel_FR_joint" type="continuous">
     <axis xyz="0 0 -1" />
-    <origin xyz="0.2 -0.2 0.05" rpy="${PI/2.0} 0 0"/>
+    <origin xyz="0.2 -0.4 0.05" rpy="${PI/2.0} 0 0"/>
     <parent link="base_link"/>
     <child link="wheel_FR_link"/>
@@ -63,13 +142,13 @@
       <origin xyz="0 0 0" rpy="0 0 0"/>
       <geometry>
-        <mesh filename="package://ngws_description/meshes/chelun.stl" scale="0.001 0.001 0.001"/>
-      </geometry>
-    </collision>
-    <visual>
-      <origin xyz="0 0 0" rpy="0 0 0"/>
-      <geometry>
-        <mesh filename="package://ngws_description/meshes/chelun.stl" scale="0.001 0.001 0.001"/>
-      </geometry>
-      <material name="black"/>
+        <mesh filename="package://ngws_description/meshes/mecanum_wheel.stl" scale="0.001 0.001 0.001"/>
+      </geometry>
+    </collision>
+    <visual>
+      <origin xyz="0 0 0" rpy="0 0 0"/>
+      <geometry>
+        <mesh filename="package://ngws_description/meshes/mecanum_wheel.stl" scale="0.001 0.001 0.001"/>
+      </geometry>
+      <material name="red"/>
     </visual>
     <inertial>
@@ -81,7 +160,7 @@
         izz="0.009"/>
     </inertial>
-  </link>
+  </link> -->
   <!-- Wheel FL -->
-  <joint name="wheel_FL_joint" type="continuous">
+  <!-- <joint name="wheel_FL_joint" type="continuous">
     <axis xyz="0 0 -1" />
     <origin xyz="0.2 0.2 0.05" rpy="${PI/2.0} 0 0"/>
@@ -93,11 +172,11 @@
       <origin xyz="0 0 0" rpy="0 0 0"/>
       <geometry>
-        <mesh filename="package://ngws_description/meshes/chelun.stl" scale="0.001 0.001 0.001"/>
-      </geometry>
-    </collision>
-    <visual>
-      <origin xyz="0 0 0" rpy="0 0 0"/>
-      <geometry>
-        <mesh filename="package://ngws_description/meshes/chelun.stl" scale="0.001 0.001 0.001"/>
+        <mesh filename="package://ngws_description/meshes/mecanum_wheel.stl" scale="0.001 0.001 0.001"/>
+      </geometry>
+    </collision>
+    <visual>
+      <origin xyz="0 0 0" rpy="0 0 0"/>
+      <geometry>
+        <mesh filename="package://ngws_description/meshes/mecanum_wheel.stl" scale="0.001 0.001 0.001"/>
       </geometry>
       <material name="black"/>
@@ -111,7 +190,7 @@
         izz="0.009"/>
     </inertial>
-  </link>
+  </link> -->
 <!-- Wheel BR -->
-  <joint name="wheel_BR_joint" type="continuous">
+ <!--  <joint name="wheel_BR_joint" type="continuous">
     <axis xyz="0 0 -1" />
     <origin xyz="-0.2 -0.2 0.05" rpy="${PI/2.0} 0 0"/>
@@ -123,11 +202,11 @@
       <origin xyz="0 0 0" rpy="0 0 0"/>
       <geometry>
-        <mesh filename="package://ngws_description/meshes/chelun.stl" scale="0.001 0.001 0.001"/>
-      </geometry>
-    </collision>
-    <visual>
-      <origin xyz="0 0 0" rpy="0 0 0"/>
-      <geometry>
-        <mesh filename="package://ngws_description/meshes/chelun.stl" scale="0.001 0.001 0.001"/>
+        <mesh filename="package://ngws_description/meshes/mecanum_wheel.stl" scale="0.001 0.001 0.001"/>
+      </geometry>
+    </collision>
+    <visual>
+      <origin xyz="0 0 0" rpy="0 0 0"/>
+      <geometry>
+        <mesh filename="package://ngws_description/meshes/mecanum_wheel.stl" scale="0.001 0.001 0.001"/>
       </geometry>
       <material name="black"/>
@@ -141,7 +220,7 @@
         izz="0.009"/>
     </inertial>
-  </link>
+  </link> -->
 <!-- Wheel BL -->
-  <joint name="wheel_BL_joint" type="continuous">
+  <!-- <joint name="wheel_BL_joint" type="continuous">
     <axis xyz="0 0 -1" />
     <origin xyz="-0.2 0.2 0.05" rpy="${PI/2.0} 0 0"/>
@@ -153,11 +232,11 @@
       <origin xyz="0 0 0" rpy="0 0 0"/>
       <geometry>
-        <mesh filename="package://ngws_description/meshes/chelun.stl" scale="0.001 0.001 0.001"/>
-      </geometry>
-    </collision>
-    <visual>
-      <origin xyz="0 0 0" rpy="0 0 0"/>
-      <geometry>
-        <mesh filename="package://ngws_description/meshes/chelun.stl" scale="0.001 0.001 0.001"/>
+        <mesh filename="package://ngws_description/meshes/mecanum_wheel.stl" scale="0.001 0.001 0.001"/>
+      </geometry>
+    </collision>
+    <visual>
+      <origin xyz="0 0 0" rpy="0 0 0"/>
+      <geometry>
+        <mesh filename="package://ngws_description/meshes/mecanum_wheel.stl" scale="0.001 0.001 0.001"/>
       </geometry>
       <material name="black"/>
@@ -171,7 +250,7 @@
         izz="0.009"/>
     </inertial>
-  </link>
+  </link> -->
   <!-- Laser -->
-  <joint name="laser_joint" type="fixed">
+ <!--  <joint name="laser_joint" type="fixed">
     <axis xyz="0 1 0" />
     <origin xyz="0.0 0 0.35" rpy="0 0 0"/>
@@ -197,5 +276,5 @@
       <inertia ixx="1e-6" ixy="0" ixz="0" iyy="1e-6" iyz="0" izz="1e-6" />
     </inertial>
-  </link>
+  </link> -->
   <joint name="camera_joint" type="fixed">
     <axis xyz="0 1 0" />
