Commit message: gazebo-7 supported

File: ngws_description/urdf/mecanum_wheel/mecanum_wheel.xacro (robot description, xacro)
@@ -12,6 +12,6 @@
         <origin xyz="0 0 0" rpy="0 ${PI/2.0} 0"/>
         <geometry>
-         <!--  <cylinder length="0.02" radius="0.03"/> -->
-          <mesh filename="${main_mesh_file}" scale="${mesh_scale} ${mesh_scale} ${mesh_scale}"/>
+          <cylinder length="0.02" radius="0.03"/>
+          <!-- <mesh filename="${main_mesh_file}" scale="${mesh_scale} ${mesh_scale} ${mesh_scale}"/> -->
         </geometry>
       </collision>

Commit message: almost fixed drifting

File: ngws_description/urdf/mecanum_wheel/mecanum_wheel.xacro (robot description, xacro)
@@ -2,6 +2,6 @@
 <robot xmlns:xacro="http://ros.org/wiki/xacro">
   <xacro:macro name="mecanum_wheel_macro"
-    params="name parent_link has_8_subwheel:=false has_10_subwheel:=false main_radius caster main_mesh_file sub_mesh_file mesh_scale mass x y z R P Y">
-		<joint name="${name}_joint" type="continuous">
+    params="name parent_link joint_type has_8_subwheel:=false has_10_subwheel:=false main_radius caster main_mesh_file sub_mesh_file mesh_scale mass x y z R P Y">
+		<joint name="${name}_joint" type="${joint_type}">
 	    <origin xyz="${x} ${y} ${z}" rpy="${R} ${P} ${Y}" />
 	    <parent link="${parent_link}" />

File: ngws_description/urdf/ngws_v1.0.xacro (robot description, xacro)
@@ -4,5 +4,5 @@
   <!-- Constants for robot dimensions -->
   <xacro:property name="PI" value="3.1415926535897931"/>
-  <xacro:property name="mass" value="60" /> <!-- arbitrary value for mass -->
+  <xacro:property name="mass" value="40" /> <!-- arbitrary value for mass -->
   <xacro:property name="width" value="0.6" /> <!-- Square dimensions (widthxwidth) of beams -->
   <!-- Import all Gazebo-customization elements, including Gazebo colors -->
@@ -148,14 +148,16 @@
   </link>
   <!-- subwheel -->
-    <xacro:property name="wheel_mass" value="5"/>
+    <xacro:property name="wheel_mass" value="2"/>
     <xacro:property name="main_radius" value="0.041"/>
     <xacro:property name="caster" value="${PI*0.25}"/>
     <xacro:property name="main_mesh_file" value="package://ngws_description/meshes/mecanum_wheel.stl"/>
     <xacro:property name="main_mesh_file_rev" value="package://ngws_description/meshes/mecanum_wheel_r.stl"/>
-    <xacro:property name="sub_mesh_file" value="package://ngws_description/meshes/mecanum_miniwheel.stl"/>
+    <xacro:property name="sub_mesh_file" value="package://ngws_description/meshes/mecanum_miniwheel_small.stl"/>
+    <xacro:property name="wheel_T_offset" value="${PI/100*0}"/>
   <!-- FR -->
   <xacro:mecanum_wheel_macro
     name="wheel_FR"
     parent_link="bridge1_link"
+    joint_type="continuous"
     mass="${wheel_mass}"
     has_10_subwheel="true"
@@ -168,5 +170,5 @@
     y="-0.3"
     z="0.02"
-    R="0.0"
+    R="${wheel_T_offset}"
     P="0.0"
     Y="${PI/2}"
@@ -177,4 +179,5 @@
     name="wheel_FL"
     parent_link="bridge2_link"
+    joint_type="continuous"
     mass="${wheel_mass}"
     has_10_subwheel="true"
@@ -187,5 +190,5 @@
     y="0.3"
     z="0.02"
-    R="0.0"
+    R="${wheel_T_offset}"
     P="0.0"
     Y="${PI/2}"
@@ -196,4 +199,5 @@
     name="wheel_BR"
     parent_link="bridge2_link"
+    joint_type="continuous"
     mass="${wheel_mass}"
     has_10_subwheel="true"
@@ -206,5 +210,5 @@
     y="-0.3"
     z="0.02"
-    R="0.0"
+    R="${wheel_T_offset}"
     P="0.0"
     Y="${PI/2}"
@@ -215,4 +219,5 @@
     name="wheel_BL"
     parent_link="bridge1_link"
+    joint_type="continuous"
     mass="${wheel_mass}"
     has_10_subwheel="true"
@@ -225,5 +230,5 @@
     y="0.3"
     z="0.02"
-    R="0.0"
+    R="${wheel_T_offset}"
     P="0.0"
     Y="${PI/2}"
